File: BM32/BM32.kicad_pcb (KiCad board)
At the start: 4 copper layers, 91.1 x 94 mm, 219 parts, among them J1 Conn_02x10_Odd_Even, J11 Conn_02x05_Odd_Even, J12 Conn_01x03, J2 Conn_01x03, J3 USB_C_Receptacle_USB2.0, J4 2x6P 2.54mm 弯针 母座, J5 USB_C_Receptacle_USB2.0, J6 2x6P 2.54mm 弯针 母座, J7 XUNPU-TF-115, J8 USB_A, J9 RJ45_HR911105a, SW1 SW_Push, SW2 SW_Push, U1 BM32F100, U10 USB3315, U11 SY6280, U12 LAN8720A, U14 SN65HVD7x, U2 MT48LC16M16A2TG, U3 MT48LC16M16A2TG, U4 HX811T, U5 EA3036, U6 XC6209B182MR, U7 HX811T, U8 CH340E, X1 OXETGLJANF-25MHZ, X2 OXETGLJANF-24MHZ, X3 OXETGLJANF-25MHZ

Commit message: Update
Parts:
- removed R61: 2.2k, lc:0402_R
- removed R88: 3.3k, lc:0402_R
- added R37: 3.3k, lc:0402_R, F.Cu at (141.4, 110.0)
- added R53: 10k, lc:0402_R, F.Cu at (137.4, 117.7)
- added SW3: SW_Push, Button_Switch_SMD:SW_Push_SPST_NO_Alps_SKRK, F.Cu at (139.2, 120.1)
- R60: value DNP -> 10k
- moved R87 6.79 mm to (140.2, 112.5), turned to 180 degrees
- moved D25 5.19 mm to (138.6, 110.1), turned to 0 degrees
- moved R89 4.90 mm to (139.6, 117.7)
- moved SW2 1.31 mm to (139.2, 124.8)
- moved D24 0.62 mm to (138.6, 114.7), turned to 0 degrees
Connections:
- D25 pad 1: Net-(D25-Pad1) -> Net-(U1-Pad103)
- U1 pad 103: GPIO0 -> Net-(U1-Pad103)
- U1 pad 105: Net-(D25-Pad1) -> Net-(U1-Pad105)
Routing:
- net Net-(U1-Pad105): track 0.00 -> 45.9 mm, vias 0 -> 2
- net Net-(U1-Pad103): track 0.00 -> 41.5 mm, vias 0 -> 2
- net Net-(D25-Pad1): track 39.5 -> 0.00 mm, vias 2 -> 0
- net GPIO0: track 32.9 -> 0.00 mm, vias 2 -> 0
- net Net-(R89-Pad2): track 50.6 -> 61.4 mm
- net +3.3VP: track 104.7 -> 111.5 mm
- net GND: track 236.3 -> 237.6 mm, vias 187 -> 188
- net Net-(R37-Pad2): track 2.98 -> 2.08 mm
- net Net-(D24-Pad2): track 3.00 -> 2.21 mm
- net Net-(FT2-Pad2): track 19.9 -> 20.6 mm
Other:
- board text added: "GPIO0"
