File: BM32/usb.kicad_sch (KiCad schematic)
At the start: 22 parts, among them J8 USB_A, U1 BM32F100, U10 USB3315, U11 SY6280, X2 OXETGLJANF-24MHZ

Commit message: Update
Parts:
- removed R61: 2.2k, lc:0402_R, symbol Device:R
- R60: value DNP -> 10k
Changed lines of the file:
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@@
   (junction (at 209.55 55.88) (diameter 0) (color 0 0 0 0)
-  )
-  (junction (at 252.73 59.69) (diameter 0) (color 0 0 0 0)
   )
   (junction (at 173.99 71.12) (diameter 0.9144) (color 0 0 0 0)
@@
     (stroke (width 0) (type default) (color 0 0 0 0))
   )
-  (wire (pts (xy 252.73 59.69) (xy 255.27 59.69))
-    (stroke (width 0) (type default) (color 0 0 0 0))
-  )
   (wire (pts (xy 207.01 63.5) (xy 209.55 63.5))
     (stroke (width 0) (type default) (color 0 0 0 0))
@@
   (wire (pts (xy 184.15 106.68) (xy 201.93 106.68))
     (stroke (width 0) (type solid) (color 0 0 0 0))
-  )
-  (wire (pts (xy 262.89 59.69) (xy 265.43 59.69))
-    (stroke (width 0) (type default) (color 0 0 0 0))
   )
   (wire (pts (xy 201.93 125.73) (xy 215.9 125.73))
@@
     )
   )
-  (global_label "GPIO0" (shape input) (at 265.43 59.69 0) (fields_autoplaced)
-    (effects (font (size 1.27 1.27)) (justify left))
-    (property "插入图纸页参考" "${INTERSHEET_REFS}" (id 0) (at 273.5279 59.7694 0)
-      (effects (font (size 1.27 1.27)) (justify left) hide)
-    )
-  )
   (symbol (lib_id "Device:R_Small") (at 242.57 120.65 0) (mirror y) (unit 1)
     (in_bom yes) (on_board yes) (fields_autoplaced)
@@
     (in_bom yes) (on_board yes)
     (property "Reference" "R60" (id 0) (at 255.27 53.34 90))
-    (property "Value" "DNP" (id 1) (at 252.73 53.34 90)
+    (property "Value" "10k" (id 1) (at 252.73 53.34 90)
       (effects (font (size 0.8 0.8)))
     )
@@
     (pin "4")
   )
-  (symbol (lib_id "Device:R") (at 259.08 59.69 270) (unit 1)
-    (in_bom yes) (on_board yes)
-    (property "Reference" "R61" (id 0) (at 259.08 62.23 90))
-    (property "Value" "2.2k" (id 1) (at 259.08 59.69 90)
-      (effects (font (size 0.8 0.8)))
-    )
-    (property "Footprint" "lc:0402_R" (id 2) (at 259.08 57.912 90)
-      (effects (font (size 1.27 1.27)) hide)
-    )
-    (property "Datasheet" "~" (id 3) (at 259.08 59.69 0)
-      (effects (font (size 1.27 1.27)) hide)
-    )
-    (pin "1")
-    (pin "2")
-  )
   (symbol (lib_id "Device:R") (at 219.71 125.73 90) (unit 1)
